File: Starbie PCB board.kicad_pcb (KiCad board)
At the start: 2 copper layers, 108.7 x 70 mm, 12 parts, among them J1 Conn_01x04_Pin, J2 Conn_01x08_Pin, SW1 SW_Push, SW2 SW_Push, U1 XIAO-ESP32-C3-SMD, U2 DHT11

Commit message: more files
Routing:
- added copper zone on B.Cu, net GND
- added copper zone on F.Cu, net GND
Changed lines of the file:
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@@
 			(plotframeref no)
 			(mode 1)
-			(useauxorigin no)
+			(useauxorigin yes)
 			(pdf_front_fp_property_popups yes)
 			(pdf_back_fp_property_popups yes)
@@
 			(outputformat 1)
 			(mirror no)
-			(drillshape 1)
+			(drillshape 0)
 			(scaleselection 1)
-			(outputdirectory "")
+			(outputdirectory "./")
 		)
 	)
@@
 		(net "/GPIO2")
 	)
+	(zone
+		(net "GND")
+		(layers "F.Cu" "B.Cu")
+		(hatch none 0.1)
+		(connect_pads yes
+			(clearance 0)
+		)
+		(min_thickness 0.025)
+		(fill yes
+			(thermal_gap 0)
+			(thermal_bridge_width 0.05)
+			(smoothing chamfer)
+			(radius 2)
+			(island_removal_mode 0)
+		)
+		(polygon
+			(pts
+				(xy 222.5 26.5) (xy 243.5 26.5) (xy 224 94) (xy 137 94) (xy 155.5 26) (xy 210 26) (xy 210.5 43)
+				(xy 211 43.5) (xy 221.5 43.5) (xy 222.5 42.5)
+			)
+		)
+	)
 	(embedded_fonts no)
